Commit message: update

File: simulation/urdf/robot.xacro (robot description, xacro)
@@ -236,5 +236,5 @@
       <origin xyz="0 0 0" rpy="0 0 0"/>
       <geometry>
-        <mesh filename="package://fast-scnn-ros/simulation/urdf/hokuyo.dae"/>
+        <mesh filename="package://gazebo2real/simulation/urdf/hokuyo.dae"/>
       </geometry>
     </visual>
